File: ldr_ads_pcb/ldr_ads_pcb.kicad_sch (KiCad schematic)
At the start: 4 parts

Commit message: feat: ready pcb
Parts:
- added J1: Conn_01x03, Connector_PinHeader_2.54mm:PinHeader_1x03_P2.54mm_Horizontal, symbol Connector_Generic:Conn_01x03
Connections:
- net +3.3V: now also J1.3 (Pin_3)
- net GND: now also J1.2 (Pin_2)
- net out: now reaches C1.1, R3.2
- net out: now also J1.1 (Pin_1)
