File: pcb/mag.kicad_pcb (KiCad board)
At the start: 2 copper layers, 85 x 85 mm, 30 parts, among them J1 Conn_01x02, J2 Conn_01x02, J3 Conn_01x03, J4 Conn_01x03, J5 Conn_01x03, J6 Conn_01x03, J7 Conn_01x02_Pin, U1 L293, U4 L7805

Commit message: pcb change and ldr setp csv file add
Parts:
- moved D8 2.50 mm to (139.7, 133.5)
Routing:
- net /LDR.Right: track 139.0 -> 141.1 mm
- net Net-(D7-K): track 13.4 -> 14.0 mm

Commit message: fix: add test to sunsensor
Routing:
- net VCC: track 128.8 -> 125.6 mm
Other:
- board text added: "CCW"
- board text added: "CW"
Changed lines of the file:
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@@
 			(psa4output no)
 			(plot_black_and_white yes)
+			(plotinvisibletext no)
 			(sketchpadsonfab no)
 			(plotpadnumbers no)
@@
 		)
 	)
+	(gr_text "CW\n"
+		(at 136 141.5 0)
+		(layer "Cmts.User")
+		(effects
+			(font
+				(size 1 1)
+				(thickness 0.15)
+			)
+			(justify left bottom)
+		)
+	)
+	(gr_text "CCW"
+		(at 168.5 112 90)
+		(layer "Cmts.User")
+		(effects
+			(font
+				(size 1 1)
+				(thickness 0.15)
+			)
+			(justify left bottom)
+		)
+	)
+	(gr_text "CCW"
+		(at 131.5 141.5 0)
+		(layer "Cmts.User")
+		(effects
+			(font
+				(size 1 1)
+				(thickness 0.15)
+			)
+			(justify left bottom)
+		)
+	)
+	(gr_text "CW"
+		(at 168.5 107.5 90)
+		(layer "Cmts.User")
+		(effects
+			(font
+				(size 1 1)
+				(thickness 0.15)
+			)
+			(justify left bottom)
+		)
+	)
 	(dimension
 		(type orthogonal)
@@
 			(keep_text_aligned yes)
 		)
-		(gr_text "42,5"
+		(gr_text "42.5"
 			(at 175.35 121.25 90)
 			(layer "F.Fab")
@@
 			(keep_text_aligned yes)
 		)
-		(gr_text "42,5"
+		(gr_text "42.5"
 			(at 175.35 78.75 90)
 			(layer "F.Fab")
@@
 	)
 	(segment
-		(start 142.19 133.5)
-		(end 139 133.5)
-		(width 0.6)
-		(layer "B.Cu")
-		(net 6)
-	)
-	(segment
 		(start 147 77.31)
 		(end 146.73 77.04)
@@
 	)
 	(zone
-		(net 6)
-		(net_name "VCC")
-		(layer "B.Cu")
-		(name "$teardrop_padvia$")
-		(hatch full 0.1)
-		(priority 30020)
-		(attr
-			(teardrop
-				(type padvia)
-			)
-		)
-		(connect_pads yes
-			(clearance 0)
-		)
-		(min_thickness 0.0254)
-		(filled_areas_thickness no)
-		(fill yes
-			(thermal_gap 0.5)
-			(thermal_bridge_width 0.5)
-			(island_removal_mode 1)
-			(island_area_min 10)
-		)
-		(polygon
-			(pts
-				(xy 141.49 133.8) (xy 141.49 133.2) (xy 140.59 132.6) (xy 139.689 133.5) (xy 140.59 134.4)
-			)
-		)
-	)
-	(zone
 		(net 13)
 		(net_name "+5V")
@@
 	)
 	(zone
+		(net 6)
+		(net_name "VCC")
+		(layer "B.Cu")
+		(name "$teardrop_padvia$")
+		(hatch full 0.1)
+		(priority 30000)
+		(attr
+			(teardrop
+				(type padvia)
+			)
+		)
+		(connect_pads yes
+			(clearance 0)
+		)
+		(min_thickness 0.0254)
+		(filled_areas_thickness no)
+		(fill yes
+			(thermal_gap 0.5)
+			(thermal_bridge_width 0.5)
+			(island_removal_mode 1)
+			(island_area_min 10)
+		)
+		(polygon
+			(pts
+				(xy 138.365736 132.441472) (xy 137.941472 132.865736) (xy 138.79 134.031947) (xy 139.690707 133.500707)
+				(xy 139.921001 132.6)
+			)
+		)
+	)
+	(zone
 		(net 10)
 		(net_name "Net-(D7-K)")
@@
 			)
 		)
-	)
-	(zone
-		(net 6)
-		(net_name "VCC")
-		(layer "B.Cu")
-		(name "$teardrop_padvia$")
-		(hatch full 0.1)
-		(priority 30013)
-		(attr
-			(teardrop
-				(type padvia)
-			)
-		)
-		(connect_pads yes
-			(clearance 0)
-		)
-		(min_thickness 0.0254)
-		(filled_areas_thickness no)
-		(fill yes
-			(thermal_gap 0.5)
-			(thermal_bridge_width 0.5)
-			(island_removal_mode 1)
-			(island_area_min 10)
-		)
-		(polygon
-			(pts
-				(xy 138.365736 132.441472) (xy 137.941472 132.865736) (xy 138.79 134.031947) (xy 139.690707 133.500707)
-				(xy 139.921001 132.6)
-			)
-		)
